Commit message: Fold pool: widen the table in x only; refuse to start if the arm is pinned
The 0.6 x 0.7 m table reached y = +0.35, into the arm's elbow, which rests below the table top in
the home pose. Every reset knocked the arm away and it stayed pinned at the table edge: a box3-mid
policy that folds 123/128 sheets on the narrow table folded 0/128 on the wide one, and two training
arrays ran to completion without a fold. The table is now 0.6 x 0.4 m, its robot-side edge where
the narrow table's was.

Startup now holds the arm at its home pose for 30 steps with the table in place and fails if any
arm joint drifts more than 2 deg (0.00 deg on this table, 25.9 deg on the old one).

Co-Authored-By: Claude Opus 5.5 (1M context) <noreply@anthropic.com>

File: assets/urdf/table_fold_pool.urdf (robot description, URDF)
Before this commit: robot box, 1 links, 0 joints
Links:
- link box: geometry collision box size=0.6 0.4 0.3; visual box size=0.6 0.4 0.3
