Commit message: Flexiv Wuji: give the Rizon its masses, and train at SimToolReal's 24576 envs
Upstream flexiv_description's get_inertias macro writes <origin>, <mass> and <inertia> straight
under <link>, without the <inertial> element URDF requires, so every parser drops them: Isaac Sim
logged "No mass specified" for each Rizon link and used defaults, and yourdfpy read mass None.
fetch_assets.sh now wraps them, and the regenerated assets give the arm its 20.7 kg. A test checks
that every moving link has an inertial; it fails on the previous URDF. Geometry is unchanged.

The launcher defaulted to Play.yaml's 8192 envs, i.e. 2 SAPG blocks. SimToolReal's released policy
was trained at 24576 (pretrained_policy/config.yaml numEnvs) with block size 4096, the 6 blocks of
its (6, 29) sigma; minibatch 98304 and horizon 16 already matched. ENVS now defaults to 24576.

Co-Authored-By: Claude Opus 5.5 <noreply@anthropic.com>

File: assets/flexiv_wuji/flexiv_description/urdf/Rizon4s.urdf (robot description, URDF)
Before this commit: robot Rizon4s, 10 links, 9 joints
Links:
- link base_link: mass None -> 3.788
- link link1: mass None -> 3.596
- link link2: mass None -> 2.69
- link link3: mass None -> 2.354
- link link4: mass None -> 2.354
- link link5: mass None -> 2.31
- link link6: mass None -> 2.223
- link link7: mass None -> 1.403

File: assets/flexiv_wuji/rizon4s_left_wuji.urdf (robot description, URDF)
Before this commit: robot rizon4s_left_wuji, 41 links, 40 joints
Links:
- link base_link: mass None -> 3.788
- link link1: mass None -> 3.596
- link link2: mass None -> 2.69
- link link3: mass None -> 2.354
- link link4: mass None -> 2.354
- link link5: mass None -> 2.31
- link link6: mass None -> 2.223
- link link7: mass None -> 1.403
